File: top/Pinky3Opt.kicad_sch (KiCad schematic)
At the start: 146 parts, among them J1 USB_C_Receptacle_USB2.0, J2 Conn_01x04, J3 USB_C_Receptacle_USB2.0, J4 Conn_01x04, SW1 Reset, SW2 Reset, U1 ATmega32U4-A, U2 PRTR5V0U2X, U3 ATmega32U4-A, U4 PRTR5V0U2X, Y1 16MHz, Y2 16MHz

Commit message: remove parts from top plate
Parts:
- removed C1, C16: 1uF, Capacitor_SMD:C_0805_2012Metric, symbol Device:C_Small
- removed C10, C13, C14, C2, C3, C4, C5, C9: 0.1uF, Capacitor_SMD:C_0805_2012Metric, symbol Device:C_Small
- removed C11, C12, C6, C7: 22pF, Capacitor_SMD:C_0805_2012Metric, symbol Device:C_Small
- removed C15, C8: 10uF, Capacitor_SMD:C_0805_2012Metric, symbol Device:C_Small
- removed D1, D10, D11, D12, D13, D14, D15, D16, D17, D18, D19, D2, D20, D21, D22, D23, D24, D25, D26, D27, D28, D29, D3, D30, D31, D32, D33, D34, D35, D36, D37, D38, D39, D4, D40, D41, D42, D43, D44, D45, D46, D47, D48, D49, D5, D50, D6, D7, D8, D9: D, Diode_SMD:D_SOD-123, symbol Device:D
- removed D61, D62: D_Schottky, Diode_SMD:D_SOD-123, symbol Device:D_Schottky
- removed F1, F2: 500mA, Fuse:Fuse_1206_3216Metric, symbol Device:Polyfuse
- removed J1, J3: USB_C_Receptacle_USB2.0, Connector_USB:USB_C_Receptacle_HRO_TYPE-C-31-M-12, symbol Connector:USB_C_Receptacle_USB2.0
- removed J2, J4: Conn_01x04, random-keyboard-parts:PJ-3200B-4A-Assembly, symbol Connector_Generic:Conn_01x04
- removed MX1, MX10, MX11, MX12, MX13, MX14, MX15, MX16, MX17, MX18, MX19, MX2, MX20, MX21, MX26, MX27, MX28, MX29, MX3, MX30, MX31, MX32, MX33, MX34, MX35, MX36, MX37, MX38, MX39, MX4, MX40, MX41, MX42, MX43, MX44, MX45, MX46, MX5, MX6, MX7, MX8, MX9: MX-NoLED, kbd:CherryMX_Hotswap, symbol MX_Alps_Hybrid:MX-NoLED
- removed MX22, MX23, MX24, MX25, MX47, MX48, MX49, MX50: MX-NoLED, kbd:ChocV1_V2_Hotswap, symbol MX_Alps_Hybrid:MX-NoLED
- removed R1, R16, R4, R9: 10kΩ, Resistor_SMD:R_0805_2012Metric, symbol Device:R_Small
- removed R10, R11, R2, R3: 22Ω, Resistor_SMD:R_0805_2012Metric, symbol Device:R_Small
- removed R12, R13, R5, R6: 5.1kΩ, Resistor_SMD:R_0805_2012Metric, symbol Device:R_Small
- removed R7, R8: 4.7kΩ, Resistor_SMD:R_0805_2012Metric, symbol Device:R_Small
- removed SW1, SW2: Reset, random-keyboard-parts:SKQGADE010, symbol Switch:SW_Push
- removed U1, U3: ATmega32U4-A, Package_QFP:TQFP-44_10x10mm_P0.8mm, symbol MCU_Microchip_ATmega:ATmega32U4-A
- removed U2, U4: PRTR5V0U2X, random-keyboard-parts:SOT143B, symbol random-keyboard-parts:PRTR5V0U2X
- removed Y1, Y2: 16MHz, Crystal:Crystal_SMD_3225-4Pin_3.2x2.5mm, symbol Device:Crystal_GND24_Small
Connections:
- no-connect marks 28 -> 0
