File: pcb/Pinky3Opt.kicad_pcb (KiCad board)
At the start: 2 copper layers, 136 x 102.7 mm, 78 parts, among them J1 USB_C_Receptacle_USB2.0, J2 Conn_01x04, SW1 Reset, U1 ATmega32U4-A, U2 PRTR5V0U2X, Y1 16MHz

Commit message: maybe done right hand
Parts:
- added ?: Val**, kbd:M2_HOLE_v2, F.Cu at (285.8, 95.2)
- added ?: Val**, kbd:M2_HOLE_v2, F.Cu at (190.5, 71.5)
- added ?: Val**, kbd:M2_HOLE_v2, F.Cu at (276.2, 113.4)
- added C10: 0.1uF, Capacitor_SMD:C_0805_2012Metric, B.Cu at (231.1, 95.7)
- added C11: 22pF, Capacitor_SMD:C_0805_2012Metric, B.Cu at (232.9, 114.4)
- added C12: 22pF, Capacitor_SMD:C_0805_2012Metric, B.Cu at (239.9, 114.4)
- added C13: 0.1uF, Capacitor_SMD:C_0805_2012Metric, B.Cu at (238.9, 95.7)
- added C14: 0.1uF, Capacitor_SMD:C_0805_2012Metric, B.Cu at (227.6, 108.0)
- added C15: 10uF, Capacitor_SMD:C_0805_2012Metric, B.Cu at (243.5, 99.1)
- added C16: 1uF, Capacitor_SMD:C_0805_2012Metric, B.Cu at (245.9, 103.9)
- added C9: 0.1uF, Capacitor_SMD:C_0805_2012Metric, B.Cu at (243.6, 111.7)
- added D26: D, Diode_SMD:D_SOD-123, B.Cu at (192.1, 64.9)
- added D27: D, Diode_SMD:D_SOD-123, B.Cu at (207.9, 64.9)
- added D28: D, Diode_SMD:D_SOD-123, B.Cu at (211.2, 64.9)
- added D29: D, Diode_SMD:D_SOD-123, B.Cu at (246.0, 60.1)
- added D30: D, Diode_SMD:D_SOD-123, B.Cu at (249.3, 60.1)
- added D31: D, Diode_SMD:D_SOD-123, B.Cu at (284.1, 69.7)
- added D32: D, Diode_SMD:D_SOD-123, B.Cu at (287.4, 69.7)
- added D33: D, Diode_SMD:D_SOD-123, B.Cu at (192.1, 88.7)
- added D34: D, Diode_SMD:D_SOD-123, B.Cu at (207.9, 83.9)
- added D35: D, Diode_SMD:D_SOD-123, B.Cu at (211.2, 83.9)
- added D36: D, Diode_SMD:D_SOD-123, B.Cu at (246.0, 79.2)
- added D37: D, Diode_SMD:D_SOD-123, B.Cu at (249.3, 79.2)
- added D38: D, Diode_SMD:D_SOD-123, B.Cu at (284.1, 88.7)
- added D39: D, Diode_SMD:D_SOD-123, B.Cu at (287.4, 88.7)
- added D40: D, Diode_SMD:D_SOD-123, B.Cu at (192.1, 112.4)
- added D41: D, Diode_SMD:D_SOD-123, B.Cu at (207.8, 100.0)
- added D42: D, Diode_SMD:D_SOD-123, B.Cu at (211.0, 100.0)
- added D43: D, Diode_SMD:D_SOD-123, B.Cu at (243.4, 94.5)
- added D44: D, Diode_SMD:D_SOD-123, B.Cu at (247.1, 94.5)
- added D45: D, Diode_SMD:D_SOD-123, B.Cu at (284.1, 107.8)
- added D46: D, Diode_SMD:D_SOD-123, B.Cu at (287.4, 107.8)
- added D47: D, Diode_SMD:D_SOD-123, B.Cu at (192.1, 119.1)
- added D48: D, Diode_SMD:D_SOD-123, B.Cu at (207.8, 119.1)
- added D49: D, Diode_SMD:D_SOD-123, B.Cu at (211.0, 119.1)
- added D50: D, Diode_SMD:D_SOD-123, B.Cu at (225.8, 119.1)
- added D62: D_Schottky, Diode_SMD:D_SOD-123, B.Cu at (247.1, 99.7)
- added F2: 500mA, Fuse:Fuse_1206_3216Metric, B.Cu at (263.9, 65.9)
- added J3: USB_C_Receptacle_USB2.0, Connector_USB:USB_C_Receptacle_HRO_TYPE-C-31-M-12, B.Cu at (275.9, 52.4)
- added J4: Conn_01x04, random-keyboard-parts:PJ-3200B-4A-Assembly, F.Cu at (171.4, 98.6)
- added MX26: MX-NoLED, kbd:CherryMX_Hotswap, F.Cu at (181.0, 66.7)
- added MX27: MX-NoLED, kbd:CherryMX_Hotswap, F.Cu at (200.0, 61.9)
- added MX28: MX-NoLED, kbd:CherryMX_Hotswap, F.Cu at (219.1, 57.1)
- added MX29: MX-NoLED, kbd:CherryMX_Hotswap, F.Cu at (238.1, 52.4)
- added MX30: MX-NoLED, kbd:CherryMX_Hotswap, F.Cu at (257.2, 57.1)
- added MX31: MX-NoLED, kbd:CherryMX_Hotswap, F.Cu at (276.2, 66.7)
- added MX32: MX-NoLED, kbd:CherryMX_Hotswap, F.Cu at (295.3, 66.7)
- added MX33: MX-NoLED, kbd:CherryMX_Hotswap, F.Cu at (181.0, 85.7)
- added MX34: MX-NoLED, kbd:CherryMX_Hotswap, F.Cu at (200.0, 81.0)
- added MX35: MX-NoLED, kbd:CherryMX_Hotswap, F.Cu at (219.1, 76.2)
- added MX36: MX-NoLED, kbd:CherryMX_Hotswap, F.Cu at (238.1, 71.4)
- added MX37: MX-NoLED, kbd:CherryMX_Hotswap, F.Cu at (257.2, 76.2)
- added MX38: MX-NoLED, kbd:CherryMX_Hotswap, F.Cu at (276.2, 85.7)
- added MX39: MX-NoLED, kbd:CherryMX_Hotswap, F.Cu at (295.3, 85.7)
- added MX40: MX-NoLED, kbd:CherryMX_Hotswap, F.Cu at (181.2, 113.8)
- added MX41: MX-NoLED, kbd:CherryMX_Hotswap, F.Cu at (200.0, 100.0)
- added MX42: MX-NoLED, kbd:CherryMX_Hotswap, F.Cu at (219.1, 95.2)
- added MX43: MX-NoLED, kbd:CherryMX_Hotswap, F.Cu at (238.1, 90.5)
- added MX44: MX-NoLED, kbd:CherryMX_Hotswap, F.Cu at (257.2, 95.2)
- added MX45: MX-NoLED, kbd:CherryMX_Hotswap, F.Cu at (276.2, 104.8)
- added MX46: MX-NoLED, kbd:CherryMX_Hotswap, F.Cu at (295.3, 104.8)
- added MX47: MX-NoLED, kbd:ChocV1_V2_Hotswap, F.Cu at (181.5, 134.6)
- added MX48: MX-NoLED, kbd:ChocV1_V2_Hotswap, F.Cu at (198.1, 126.8)
- added MX49: MX-NoLED, kbd:ChocV1_V2_Hotswap, F.Cu at (215.9, 122.0)
- added MX50: MX-NoLED, kbd:ChocV1_V2_Hotswap, F.Cu at (234.4, 120.4)
- added R10: 22, Resistor_SMD:R_0805_2012Metric, B.Cu at (257.2, 102.1)
- added R11: 22, Resistor_SMD:R_0805_2012Metric, B.Cu at (257.2, 104.5)
- added R12: 5.1k, Resistor_SMD:R_0805_2012Metric, B.Cu at (285.7, 60.6)
- added R13: 5.1k, Resistor_SMD:R_0805_2012Metric, B.Cu at (285.7, 57.6)
- added R16: 10k, Resistor_SMD:R_0805_2012Metric, B.Cu at (225.2, 108.0)
- added R4: 10k, Resistor_SMD:R_0805_2012Metric, B.Cu at (226.9, 99.4)
- added Ref**: Val**, kbd:M2_HOLE_v2, F.Cu at (285.8, 71.4)
- added SW2: Reset, random-keyboard-parts:SKQGADE010, B.Cu at (257.2, 110.4)
- added U3: ATmega32U4-A, Package_QFP:TQFP-44_10x10mm_P0.8mm, B.Cu at (235.8, 103.8)
- added U4: PRTR5V0U2X, random-keyboard-parts:SOT143B, B.Cu at (266.2, 60.5)
- added Y2: 16MHz, Crystal:Crystal_SMD_3225-4Pin_3.2x2.5mm, B.Cu at (236.4, 114.4)
- moved D14 21.7 mm to (141.2, 88.7)
- moved C6 21.4 mm to (101.8, 96.5)
- moved ? 21.4 mm to (133.3, 113.4)
- moved C1 21.4 mm to (89.2, 106.9)
- moved C4 21.4 mm to (103.1, 115.4)
- moved C8 21.4 mm to (87.3, 100.0)
- moved D10 21.4 mm to (84.1, 79.2)
- moved D11 21.4 mm to (87.3, 79.2)
- moved D12 21.4 mm to (122.2, 83.9)
- moved D13 21.4 mm to (125.5, 83.9)
- moved D20 21.4 mm to (122.2, 100.0)
- moved D22 21.4 mm to (107.6, 119.1)
- moved D23 21.4 mm to (122.2, 119.1)
- moved D24 21.4 mm to (125.5, 119.1)
- moved D25 21.4 mm to (141.2, 119.1)
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- renumbered D26 to D61
Connections:
- net /D+ renamed /D+_L
- net /D- renamed /D-_L
- net /SCL renamed /SCL_L
- net /SDA renamed /SDA_L
Routing:
- net GNDA: track 0.00 -> 270.1 mm
- net /ROW0_R: track 0.00 -> 185.8 mm, vias 0 -> 4
- net /ROW1_R: track 0.00 -> 161.4 mm, vias 0 -> 4
- net /ROW2_R: track 0.00 -> 141.4 mm, vias 0 -> 5
- net /COL0_R: track 0.00 -> 129.2 mm, vias 0 -> 5
- net /COL1_R: track 0.00 -> 118.5 mm, vias 0 -> 5
- net +5VA: track 0.00 -> 108.3 mm, vias 0 -> 6
- net /COL3_R: track 0.00 -> 104.7 mm, vias 0 -> 5
- net /COL2_R: track 0.00 -> 94.8 mm, vias 0 -> 5
- net /COL6_R: track 0.00 -> 90.2 mm, vias 0 -> 4
- net /COL5_R: track 0.00 -> 67.8 mm, vias 0 -> 4
- net /SCL_R: track 0.00 -> 65.2 mm, vias 0 -> 2
- net Net-(U4-IO1): track 0.00 -> 64.2 mm
- net Net-(U4-IO2): track 0.00 -> 62.3 mm
- net VDC: track 0.00 -> 61.0 mm, vias 0 -> 2
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- added copper zone on B.Cu, net GNDA
Other:
- board size 136 x 102.7 mm -> 276.2 x 102.7 mm

Commit message: breakaway
Parts:
- added REF**: breakaway-mousebites, random-keyboard-parts:breakaway-mousebites, F.Cu at (257.2, 114.3)
- added REF**: breakaway-mousebites, random-keyboard-parts:breakaway-mousebites, F.Cu at (95.2, 42.9)
- added REF**: breakaway-mousebites, random-keyboard-parts:breakaway-mousebites, F.Cu at (38.1, 114.3)
- added REF**: breakaway-mousebites, random-keyboard-parts:breakaway-mousebites, F.Cu at (295.3, 114.3)
- added REF**: breakaway-mousebites, random-keyboard-parts:breakaway-mousebites, F.Cu at (238.1, 42.9)
- added REF**: breakaway-mousebites, random-keyboard-parts:breakaway-mousebites, F.Cu at (76.2, 114.3)
Other:
- board size 276.2 x 102.7 mm -> 276.2 x 126 mm

Commit message: silkscreen
Parts:
- moved R13 0.61 mm to (285.9, 58.2)
- moved R12 0.22 mm to (285.9, 60.5)
Routing:
- net GNDA: track 270.1 -> 269.3 mm

Commit message: tweak
Routing:
- net Net-(D21-A): track 22.4 -> 25.2 mm
- net /COL2_R: track 94.8 -> 94.0 mm
- net Net-(U3-XTAL2): track 9.52 -> 9.00 mm

Commit message: jlcpcb pcba configuration
Parts:
- R1, R16, R4, R9: value 10k -> 10kΩ
- R10, R11, R2, R3: value 22 -> 22Ω
- R12, R13, R5, R6: value 5.1k -> 5.1kΩ
- R7, R8: value 4.7k -> 4.7kΩ

Commit message: tweak
Parts:
- removed ? (x6): Val**, kbd:M2_HOLE_v2
- removed the Ref** at (285.8, 71.4)
- added Ref**: Val**, kbd_Hole:m2_Spacer_Hole, F.Cu at (285.8, 95.2)
- added Ref**: Val**, kbd_Hole:m2_Spacer_Hole, F.Cu at (190.5, 71.5)
- added Ref**: Val**, kbd_Hole:m2_Spacer_Hole, F.Cu at (47.6, 95.2)
- added Ref**: Val**, kbd_Hole:m2_Spacer_Hole, F.Cu at (133.3, 113.4)
- added Ref**: Val**, kbd_Hole:m2_Spacer_Hole, F.Cu at (200.0, 113.4)
- added Ref**: Val**, kbd_Hole:m2_Spacer_Hole, F.Cu at (47.6, 76.2)
- added Ref**: Val**, kbd_Hole:m2_Spacer_Hole, F.Cu at (285.8, 76.2)
- Ref**: footprint kbd:M2_HOLE_v2 -> kbd_Hole:m2_Spacer_Hole
- moved R7 0.63 mm to (113.0, 101.0)
Other:
- board text added: "JLCJLCJLCJLC"
- board text added: "Pinky3 Opt v0.1"

Commit message: silk
Other:
- board text added: "Pinky3 Opt v0.1 designed by @tamanishi"
- board text removed: "Pinky3 Opt v0.1"
