File: pcb/Pinky3Opt.kicad_sch (KiCad schematic)
At the start: 74 parts, among them J1 USB_C_Receptacle_USB2.0, J2 Conn_01x04, SW1 Reset, U1 ATmega32U4-A, U2 PRTR5V0U2X, Y1 16MHz

Commit message: maybe done right hand
Parts:
- added C10, C13, C14, C9: 0.1uF, Capacitor_SMD:C_0805_2012Metric, symbol Device:C_Small
- added C11, C12: 22pF, Capacitor_SMD:C_0805_2012Metric, symbol Device:C_Small
- added C15: 10uF, Capacitor_SMD:C_0805_2012Metric, symbol Device:C_Small
- added C16: 1uF, Capacitor_SMD:C_0805_2012Metric, symbol Device:C_Small
- added D26, D27, D28, D29, D30, D31, D32, D33, D34, D35, D36, D37, D38, D39, D40, D41, D42, D43, D44, D45, D46, D47, D48, D49, D50: D, Diode_SMD:D_SOD-123, symbol Device:D
- added D62: D_Schottky, Diode_SMD:D_SOD-123, symbol Device:D_Schottky
- added F2: 500mA, Fuse:Fuse_1206_3216Metric, symbol Device:Polyfuse
- added J3: USB_C_Receptacle_USB2.0, Connector_USB:USB_C_Receptacle_HRO_TYPE-C-31-M-12, symbol Connector:USB_C_Receptacle_USB2.0
- added J4: Conn_01x04, random-keyboard-parts:PJ-3200B-4A-Assembly, symbol Connector_Generic:Conn_01x04
- added MX26, MX27, MX28, MX29, MX30, MX31, MX32, MX33, MX34, MX35, MX36, MX37, MX38, MX39, MX40, MX41, MX42, MX43, MX44, MX45, MX46: MX-NoLED, kbd:CherryMX_Hotswap, symbol MX_Alps_Hybrid:MX-NoLED
- added MX47, MX48, MX49, MX50: MX-NoLED, kbd:ChocV1_V2_Hotswap, symbol MX_Alps_Hybrid:MX-NoLED
- added R10, R11: 22, Resistor_SMD:R_0805_2012Metric, symbol Device:R_Small
- added R12, R13: 5.1k, Resistor_SMD:R_0805_2012Metric, symbol Device:R_Small
- added R16, R4: 10k, Resistor_SMD:R_0805_2012Metric, symbol Device:R_Small
- added SW2: Reset, random-keyboard-parts:SKQGADE010, symbol Switch:SW_Push
- added U3: ATmega32U4-A, Package_QFP:TQFP-44_10x10mm_P0.8mm, symbol MCU_Microchip_ATmega:ATmega32U4-A
- added U4: PRTR5V0U2X, random-keyboard-parts:SOT143B, symbol random-keyboard-parts:PRTR5V0U2X
- added Y2: 16MHz, Crystal:Crystal_SMD_3225-4Pin_3.2x2.5mm, symbol Device:Crystal_GND24_Small
- renumbered D26 to D61
Connections:
- net D+ renamed D+_L
- net D- renamed D-_L
- net SCL renamed SCL_L
- net SDA renamed SDA_L
- new net: D30.2 (A), MX30.2 (ROW)
- new net: D29.2 (A), MX29.2 (ROW)
- new net: D49.2 (A), MX49.2 (ROW)
- new net: D44.2 (A), MX44.2 (ROW)
- new net: D38.2 (A), MX38.2 (ROW)
- new net: D35.2 (A), MX35.2 (ROW)
- new net: D33.2 (A), MX33.2 (ROW)
- new net: D32.2 (A), MX32.2 (ROW)
- new net: D50.2 (A), MX50.2 (ROW)
- new net: D43.2 (A), MX43.2 (ROW)
- new net: D37.2 (A), MX37.2 (ROW)
- new net: R4.1, U3.33 (~{HWB}/PE2)
- new net: D46.2 (A), MX46.2 (ROW)
- new net: D45.2 (A), MX45.2 (ROW)
- new net: D31.2 (A), MX31.2 (ROW)
- new net: C12.2, U3.16 (XTAL2), Y2.3
- new net: D40.2 (A), MX40.2 (ROW)
- new net: D34.2 (A), MX34.2 (ROW)
- new net: J3.A5 (CC1), R12.1
- new net: J3.A6 (D+), J3.B6 (D+), R11.1, U4.2 (IO1)
- new net: J3.A7 (D-), J3.B7 (D-), R10.1, U4.3 (IO2)
- new net: J3.B5 (CC2), R13.1
- new net: D36.2 (A), MX36.2 (ROW)
- new net: C11.2, U3.17 (XTAL1), Y2.1
- new net: D41.2 (A), MX41.2 (ROW)
- new net: D28.2 (A), MX28.2 (ROW)
- new net: D39.2 (A), MX39.2 (ROW)
- new net: D48.2 (A), MX48.2 (ROW)
- new net: D26.2 (A), MX26.2 (ROW)
- new net: D42.2 (A), MX42.2 (ROW)
- new net: SW2.2, U3.13 (~{RESET})
- new net: C16.1, U3.6 (UCAP)
- new net: D27.2 (A), MX27.2 (ROW)
- new net: D47.2 (A), MX47.2 (ROW)
- new net +5VA: C10.1, C13.1, C14.1, C9.1, D62.1 (K), J4.4 (Pin_4), U3.14 (VCC), U3.24 (AVCC), U3.34 (VCC), U3.44 (AVCC)
- new net COL0_R: MX26.1 (COL), MX33.1 (COL), MX40.1 (COL), MX47.1 (COL), U3.29 (PB5)
- new net COL1_R: MX27.1 (COL), MX34.1 (COL), MX41.1 (COL), MX48.1 (COL), U3.28 (PB4)
- new net COL2_R: MX28.1 (COL), MX35.1 (COL), MX42.1 (COL), MX49.1 (COL), U3.27 (PD7)
- new net COL3_R: MX29.1 (COL), MX36.1 (COL), MX43.1 (COL), MX50.1 (COL), U3.26 (PD6)
- new net COL4_R: MX30.1 (COL), MX37.1 (COL), MX44.1 (COL), U3.9 (PB1)
- new net COL5_R: MX31.1 (COL), MX38.1 (COL), MX45.1 (COL), U3.10 (PB2)
- new net COL6_R: MX32.1 (COL), MX39.1 (COL), MX46.1 (COL), U3.11 (PB3)
- new net D+_R: R11.2, U3.4 (D+)
- new net D-_R: R10.2, U3.3 (D-)
- new net GNDA: C10.2, C11.1, C12.1, C13.2, C14.2, C15.2, C16.2, C9.2, J3.A1 (GND), J3.A12 (GND), J3.B1 (GND), J3.B12 (GND), J3.S1 (SHIELD), J4.1 (Pin_1), R12.2, R13.2, R16.2, R4.2, SW2.1, U3.15 (GND), U3.23 (GND), U3.35 (GND), U3.43 (GND), U3.5 (UGND), U4.1 (GND), Y2.2, Y2.4
- new net HDETECT_R: R16.1, U3.22 (PD5)
- new net ROW0_R: D26.1 (K), D27.1 (K), D28.1 (K), D29.1 (K), D30.1 (K), D31.1 (K), D32.1 (K), U3.30 (PB6)
- new net ROW1_R: D33.1 (K), D34.1 (K), D35.1 (K), D36.1 (K), D37.1 (K), D38.1 (K), D39.1 (K), U3.31 (PC6)
- new net ROW2_R: D40.1 (K), D41.1 (K), D42.1 (K), D43.1 (K), D44.1 (K), D45.1 (K), D46.1 (K), U3.32 (PC7)
- new net ROW3_R: D47.1 (K), D48.1 (K), D49.1 (K), D50.1 (K), U3.25 (PD4)
- new net SCL_R: J4.2 (Pin_2), U3.18 (PD0)
- new net SDA_R: J4.3 (Pin_3), U3.19 (PD1)
- new net VDC: C15.1, D62.2 (A), F2.2, U3.2 (UVCC), U3.7 (VBUS)
- new net VDD: F2.1, J3.A4 (VBUS), J3.A9 (VBUS), J3.B4 (VBUS), J3.B9 (VBUS), U4.4 (VCC)
- no-connect marks 14 -> 28

Commit message: jlcpcb pcba configuration
Parts:
- C1, C16: LCSC (none) -> C28323
- C10, C13, C14, C2, C3, C4, C5, C9: LCSC (none) -> C49678
- C11, C12, C6, C7: LCSC (none) -> C1804
- C15, C8: LCSC (none) -> C15850
- D1, D10, D11, D12, D13, D14, D15, D16, D17, D18, D19, D2, D20, D21, D22, D23, D24, D25, D26, D27, D28, D29, D3, D30, D31, D32, D33, D34, D35, D36, D37, D38, D39, D4, D40, D41, D42, D43, D44, D45, D46, D47, D48, D49, D5, D50, D6, D7, D8, D9: LCSC (none) -> C81598
- D61, D62: LCSC (none) -> C162059
- F1, F2: LCSC (none) -> C369159
- J1, J3: LCSC (none) -> C165948
- R1, R16, R4, R9: value 10k -> 10kΩ; LCSC (none) -> C17414
- R10, R11, R2, R3: value 22 -> 22Ω; LCSC (none) -> C17561
- R12, R13, R5, R6: value 5.1k -> 5.1kΩ; LCSC (none) -> C27834
- R7, R8: value 4.7k -> 4.7kΩ; LCSC (none) -> C17673
- SW1, SW2: LCSC (none) -> C116647
- U1, U3: LCSC (none) -> C44854
- U2, U4: LCSC (none) -> C2827688
- Y1, Y2: LCSC (none) -> C13738

Commit message: tweak
Parts:
- SW1, SW2: LCSC C116647 -> C318884
Changed lines of the file:
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@@
       (effects (font (size 1.27 1.27)) hide)
     )
-    (property "LCSC" "C116647" (at 55.88 33.8328 0)
+    (property "LCSC" "C318884" (at 55.88 33.8328 0)
       (effects (font (size 1.27 1.27)) hide)
     )
@@
       (effects (font (size 1.27 1.27)) hide)
     )
-    (property "LCSC" "C116647" (at 55.7784 147.7772 0)
+    (property "LCSC" "C318884" (at 55.7784 147.7772 0)
       (effects (font (size 1.27 1.27)) hide)
     )
